Commit message: Added y position for the camera in URDF

File: urdf/sdl_robot_dual_arm.urdf.xacro (robot description, xacro)
@@ -59,9 +59,12 @@
   <!--<joint name="${prefix}camera_to_hardware" type="fixed">-->
   <joint name="camera_to_hardware" type="fixed">
-    <!--<parent link="${prefix}connecting_hardware"/>-->
     <parent link="connecting_hardware"/>
-    <!--<child link="${prefix}camera"/>-->
     <child link="${prefix}camera"/>
     <origin xyz=".5 0 .9" rpy="0 0 0"/>
   </joint>
+  <joint name="camera_to_hardware" type="fixed">
+    <parent link="connecting_hardware"/>
+    <child link="${prefix}camera"/>
+    <origin xyz="0 0.25 .9" rpy="0 0 0"/>
+  </joint>
 </robot>

Commit message: Corrected the position of the camera

File: urdf/sdl_robot_dual_arm.urdf.xacro (robot description, xacro)
@@ -58,13 +58,13 @@
   <xacro:include filename="$(find sdl_robot_description)/urdf/camera.urdf.xacro" />
   <!--<joint name="${prefix}camera_to_hardware" type="fixed">-->
+  <!-- <joint name="camera_to_hardware" type="fixed">
+    <parent link="connecting_hardware"/>
+    <child link="${prefix}camera"/>
+    <origin xyz=".5 0 .9" rpy="0 0 0"/>
+  </joint> -->
   <joint name="camera_to_hardware" type="fixed">
     <parent link="connecting_hardware"/>
     <child link="${prefix}camera"/>
-    <origin xyz=".5 0 .9" rpy="0 0 0"/>
-  </joint>
-  <joint name="camera_to_hardware" type="fixed">
-    <parent link="connecting_hardware"/>
-    <child link="${prefix}camera"/>
-    <origin xyz="0 0.25 .9" rpy="0 0 0"/>
+    <origin xyz="0 0.25 .9" rpy="0 0 1.57"/>
   </joint>
 </robot>
