Commit message: fixed issue with gripper model

File: urdf/2f140.urdf.xacro (robot description, xacro)
@@ -1,6 +1,6 @@
 <?xml version="1.0"?>
 <robot xmlns:xacro="http://ros.org/wiki/xacro" >
-  <xacro:include filename="$(find robotiq_2f_140_gripper_visualization)/urdf/robotiq_arg2f_140_model_macro.xacro" />
-  <xacro:robotiq_arg2f_140 prefix="${prefix}"/>
+  <xacro:include filename="$(find robotiq_2f_85_gripper_visualization)/urdf/robotiq_arg2f_85_model_macro.xacro" />
+  <xacro:robotiq_arg2f_85 prefix="${prefix}"/>
   <gazebo>
       <!-- loading plugin: mimic joints works in gazebo now-->

File: urdf/2f140_2.urdf.xacro (robot description, xacro)
@@ -1,6 +1,6 @@
 <?xml version="1.0"?>
 <robot xmlns:xacro="http://ros.org/wiki/xacro" >
-  <xacro:include filename="$(find robotiq_2f_140_gripper_visualization)/urdf/robotiq_arg2f_140_model_macro.xacro" />
-  <xacro:robotiq_arg2f_140 prefix="${prefix}_2"/>
+  <xacro:include filename="$(find robotiq_2f_85_gripper_visualization)/urdf/robotiq_arg2f_85_model_macro.xacro" />
+  <xacro:robotiq_arg2f_85 prefix="${prefix}_2"/>
   <gazebo>
       <!-- loading plugin: mimic joints works in gazebo now-->

File: urdf/sdl_robot_dual_arm.urdf.xacro (robot description, xacro)
@@ -66,5 +66,5 @@
     <parent link="connecting_hardware"/>
     <child link="${prefix}camera"/>
-    <origin xyz="0 0.25 .9" rpy="0 0 1.57"/>
+    <origin xyz="-0.026 0.15 .9" rpy="0 0 1.57"/>
   </joint>
 </robot>
